File: RFToy.brd (EAGLE design)
At the start: 58 x 38 mm, 33 parts, among them IC1 ATMEGA328P, IC4 CH340G, J1 AYZ0202, X1 USBSMD, X2 12MHz

Commit message: correct pin assignments
Parts:
- moved J1 4.83 mm to (54.0, 5.60), turned to 90 degrees
Connections:
- net D3: now also JP6.15; no longer S1.1, S1.2
- net D4: now also S1.1, S1.2; no longer S2.1, S2.2
- net D5: now also S2.1, S2.2; no longer JP6.15
Routing:
- net D5: track 20.8 -> 41.5 mm, vias 1 -> 3
- net D7: track 34.3 -> 22.8 mm
- net D3: track 34.1 -> 24.4 mm, vias 1 -> 3
- net VBAT: track 16.6 -> 25.3 mm
- net D4: track 27.8 -> 33.4 mm
- net VIN: track 144.5 -> 149.9 mm
- net 3.3V: track 69.7 -> 64.9 mm
- net GND: track 246.7 -> 243.1 mm
- net VCC: track 113.1 -> 110.7 mm
Other:
- board text added: "GND D10 D3"
- board text removed: "GND D10 D5"
